Commit message: Update robot description

File: turtlebot_arm_description/urdf/arm_hardware.xacro (robot description, xacro)
@@ -11,4 +11,6 @@
   <xacro:property name="AX12_LENGTH" value="0.050"/>
   <xacro:property name="F2_HEIGHT" value="0.0265"/>
+  <xacro:property name="FACTOR_GRIPPER_TRANSL" value="0.01"/>
+  <xacro:property name="OFFSET_GRIPPER_TRANSL" value="0.029"/>
   <xacro:macro name="arm_mount" params="parent name color *origin">
     <joint name="${name}_joint" type="fixed">

File: turtlebot_arm_description/urdf/pincher_arm.urdf.xacro (robot description, xacro)
@@ -22,5 +22,5 @@
       <!-- Place the "floating" arm at the location it should be if mounted on a turtlebot,
            as pick and place and other demos assume this location -->
-      <origin xyz="0.1 0.03 0.435"/>
+      <origin xyz="0 0 0"/>
     </turtlebot_arm>
 </robot>

File: turtlebot_arm_description/urdf/pincher_gripper.xacro (robot description, xacro)
@@ -10,13 +10,23 @@
     </dynamixel_AX12_fixed>
      <gripper_finger_base parent="gripper_servo_link" name="gripper_finger_base" color="${color}">
-      <origin xyz="0.01  ${AX12_WIDTH} 0" rpy="${M_PI/2} ${-M_PI} ${M_PI/2}"/>
+      <origin xyz="0.015  ${AX12_WIDTH} 0" rpy="${M_PI/2} ${-M_PI} ${M_PI/2}"/>
     </gripper_finger_base>
      <!-- Finger 1 -->
+    <!-- Modifications by C. Roesmann: Instead of changing the arbotix driver to distinguish between a prismatic and a revolute joint, we do  the conversion here using a mimic. -->
     <joint name="gripper_joint" type="prismatic">
       <origin xyz="0 0 0" rpy="0 0 0"/>
       <axis xyz="1 0 0"/>
-      <limit effort="30" velocity="0.5" lower="0.002" upper="0.031"/>
+      <limit effort="30" velocity="0.5" lower="-0.8" upper="0.8"/> <!--lower="0.002" upper="0.031"-->
+      <parent link="gripper_servo_link"/>
+      <child link="link_revolute_to_prismatic_virtual1"/>
+    </joint>
+    <link name="link_revolute_to_prismatic_virtual1"/>
+    <joint name="gripper_joint_prismatic1" type="prismatic">
+      <origin xyz="0 0 0" rpy="0 0 0"/>
+      <axis xyz="1 0 0"/>
+      <limit effort="30" velocity="0.5" lower="-1" upper="1"/>
       <parent link="gripper_servo_link"/>
       <child link="gripper_active_link"/>
+      <mimic joint="gripper_joint" multiplier="${FACTOR_GRIPPER_TRANSL}"  offset = "${OFFSET_GRIPPER_TRANSL}"/>
     </joint>
     <pincher_gripper name="gripper_active" color="${color}" >
@@ -25,10 +35,10 @@
     <!-- Finger 2 -->
     <!-- Note: currently static but should be a Mimic of Finger 1 -->
-    <joint name="gripper2_joint" type="fixed">
+    <!--joint name="gripper2_joint" type="fixed">
       <parent link="gripper_servo_link"/>
       <child link="gripper_active2_link"/>
-    </joint>
+    </joint>  -->
     <pincher_gripper name="gripper_active2" color="${color}" >
-      <origin xyz="-0.02 0.023 0" rpy="${-M_PI/2} ${M_PI} 0"/>
+      <origin xyz="0.02 0.023 0" rpy="${-M_PI/2} ${M_PI} 0"/>
     </pincher_gripper>
     <!-- Using Mimic -->
@@ -43,3 +53,12 @@
       <mimic joint="gripper_joint" multiplier="-.5"  offset = "0"/>
     </joint-->
+    <!-- Changes by C. Roesmann -->
+    <joint name="gripper2_joint" type="prismatic">
+      <origin xyz="0 0 0" rpy="0 0 0"/>
+      <axis xyz="1 0 0"/>
+      <limit effort="30" velocity="0.5" lower="-10" upper="10"/>
+      <parent link="gripper_servo_link"/>
+      <child link="gripper_active2_link"/>
+      <mimic joint="gripper_joint" multiplier="-${FACTOR_GRIPPER_TRANSL}"  offset = "-${OFFSET_GRIPPER_TRANSL}"/>
+    </joint>
 </robot>

File: turtlebot_arm_description/urdf/turtlebot_arm.urdf.xacro (robot description, xacro)
@@ -3,5 +3,5 @@
 <robot name="turtlebot_arm" xmlns:xacro="http://ros.org/wiki/xacro">
     <!-- We can configure joints velocity limit and lower/upper limits
-          to allow access to different operational areas, e.g. left handed vs. right handed robot -->
+         to allow access to different operational areas, e.g. left handed vs. right handed robot -->
     <xacro:property name="joints_vlimit" value="1.571"/>
     <xacro:property name="pan_llimit" value="-2.617"/>
@@ -11,6 +11,6 @@
     <xacro:property name="elbow_llimit" value="-2.617"/>
     <xacro:property name="elbow_ulimit" value="2.617"/>
-    <xacro:property name="wrist_llimit" value="-2.617"/>
-    <xacro:property name="wrist_ulimit" value="2.617"/>
+    <xacro:property name="wrist_llimit" value="-1.745"/>
+    <xacro:property name="wrist_ulimit" value="1.745"/>
     <!-- Included URDF Files -->
     <xacro:include filename="$(find turtlebot_arm_description)/urdf/turtlebot_arm.xacro"/>

File: turtlebot_arm_description/urdf/turtlebot_arm.xacro (robot description, xacro)
@@ -93,7 +93,7 @@
   <xacro:include filename="$(find turtlebot_arm_description)/urdf/pincher_gripper.xacro"/>
   </xacro:if>
-  <!--<xacro:if value="${turtlebot_gripper}">
+  <xacro:if value="${turtlebot_gripper}">
   <xacro:include filename="$(find turtlebot_arm_description)/urdf/turtlebot_gripper.xacro"/>
-  </xacro:if>-->
+  </xacro:if>
   </xacro:macro>
 </robot>
